File: Turn-On-Test/Turn-On-Test.sch (EAGLE design)
At the start: 0 parts

Commit message: Test schematic done
Parts:
- added J1: (no value), SparkFun-Connectors:M02PTH
- added R1, R2: (no value), SparkFun-Passives:RESISTOR0603-RES
- added U$1, U$3: 22V, MotherboardParts:ZENER-SOT23
- added U$2: 5V, MotherboardParts:ZENER-SOT23
- added U$4: NMOSFET-DPAK, MotherboardParts:NMOSFET-DPAK
Connections:
- new net GND: J1.2, R1.1, U$2.A, U$4.S
- new net N$1: U$1.C, U$3.A
- new net N$2: R1.2, U$1.A, U$4.G
- new net N$3: R2.1, U$2.C, U$4.D1
- new net V+: J1.1, R2.2, U$3.C
