File: DC-DC-Brick/DC-DC-Brick.brd (EAGLE design)
At the start: 100 x 80 mm, 22 parts

Commit message: Worked on Board Layout
Parts:
- moved C19 35.2 mm to (13.5, 63.2), turned to 180 degrees
- moved SV1 33.2 mm to (58.4, 36.8)
- moved C20 31.6 mm to (13.5, 65.8), turned to 180 degrees
- moved C16 31.6 mm to (42.9, 27.4), turned to 90 degrees
- moved JP2 31.4 mm to (27.9, 6.35)
- moved C15 29.1 mm to (40.4, 27.4), turned to 90 degrees
- moved R6 24.2 mm to (25.9, 71.1), turned to 270 degrees
- moved C14 22.4 mm to (37.8, 27.4), turned to 90 degrees
- moved R3 22.2 mm to (25.9, 61.7), turned to 90 degrees
- moved R2 22.1 mm to (30.0, 71.1), turned to 270 degrees
- moved R4 22.0 mm to (22.4, 61.7), turned to 90 degrees
- moved C21 19.0 mm to (13.5, 68.3), turned to 180 degrees
- moved R1 13.6 mm to (30.0, 62.0), turned to 180 degrees
- moved R9 12.8 mm to (32.0, 57.1), turned to 270 degrees
- moved LED2 10.4 mm to (28.4, 58.2), turned to 180 degrees
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Connections:
- removed net V+: SV1.1, SV1.39
- net +12V1: now also SV1.1, SV1.11, SV1.13, SV1.15, SV1.17, SV1.19, SV1.21, SV1.23, SV1.25, SV1.27, SV1.29, SV1.3, SV1.31, SV1.33, SV1.35, SV1.37, SV1.39, SV1.5, SV1.7, SV1.9
- net GND: now also D1.C, D2.C, SV1.10, SV1.12, SV1.14, SV1.16, SV1.18, SV1.20, SV1.22, SV1.24, SV1.26, SV1.28, SV1.30, SV1.32, SV1.34, SV1.36, SV1.38, SV1.4, SV1.6, SV1.8; no longer R3.1, R4.1
- net N$4: now also D1.A, R3.1; no longer D1.C, R3.2
- net N$5: now also D2.A, R4.1; no longer D2.C, R4.2
- net N$6: now also R4.2; no longer D2.A
- net N$7: now also R3.2; no longer D1.A
- net V-: now also SV1.44, SV1.46, SV1.48
- net VCC: now also SV1.43, SV1.45, SV1.47
Routing:
- net GND: track 0.00 -> 8.66 mm, vias 0 -> 11
- net N$12: track 0.00 -> 3.70 mm
- net N$2: track 0.00 -> 3.40 mm
- net N$3: track 0.00 -> 3.24 mm
- net N$1: track 0.00 -> 3.24 mm
- net N$6: track 0.00 -> 3.13 mm
- net N$7: track 0.00 -> 2.48 mm
- net N$5: track 0.00 -> 1.83 mm
- net N$4: track 0.00 -> 1.83 mm
- added copper zone on layer 1, net +12V1
- added copper zone on layer 1, net GND
- added copper zone on layer 16, net GND
- added copper zone on layer 1, net V-
- added copper zone on layer 16, net V-
- added copper zone on layer 1, net VCC
Other:
- board size 100 x 80 mm -> 65.2 x 80 mm

Commit message: Worked on Board Layout
Parts:
- moved R2 7.73 mm to (23.1, 67.6)
- moved R6 7.73 mm to (19.1, 67.6)
- moved C15 7.73 mm to (33.5, 23.9)
- moved C16 7.73 mm to (36.1, 23.9)
- moved JP1 7.73 mm to (49.0, 72.1)
- moved SV1 7.73 mm to (51.6, 33.3)
- moved R3 7.73 mm to (19.1, 58.2)
- moved R4 7.73 mm to (15.5, 58.2)
- moved C19 7.73 mm to (6.60, 59.7)
- moved C20 7.73 mm to (6.60, 62.2)
- moved C22V1 7.73 mm to (11.2, 28.2)
- moved C22V5 7.73 mm to (20.1, 28.2)
- moved C22V6 7.73 mm to (29.0, 28.2)
- moved JP2 7.73 mm to (21.1, 2.79)
- moved D1 7.73 mm to (19.1, 54.6)
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Other:
- board size 65.2 x 80 mm -> 57.4 x 76.2 mm

Commit message: Worked on Board Layout
Parts:
- removed JP1: (no value), pinhead:1X02
- removed JP2: (no value), pinhead:1X01
- removed SV1: (no value), con-lsta:FE25-2
- added U$2: POWERBRICKCONNECTOR, newConnector:FE25-2
- moved C14 2.29 mm to (31.0, 21.6)
- moved C15 2.29 mm to (33.5, 21.6)
- moved C16 2.29 mm to (36.1, 21.6)
- moved D1 2.29 mm to (19.1, 52.3)
- moved D2 2.29 mm to (15.5, 52.3)
- moved LED2 2.29 mm to (21.6, 52.3)
- moved R1 2.29 mm to (23.1, 56.1)
- moved R9 2.29 mm to (25.1, 51.3)
- moved U$1 2.29 mm to (21.1, 34.8)
- moved C22V1 2.29 mm to (11.2, 25.9)
- moved C22V5 2.29 mm to (20.1, 25.9)
- moved C22V6 2.29 mm to (29.0, 25.9)
- moved C19 2.29 mm to (6.60, 57.4)
- moved C20 2.29 mm to (6.60, 59.9)
- moved C21 2.29 mm to (6.60, 62.5)
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Connections:
- removed net N$10: JP1.2, U$1.11
- new net N$8: U$1.11, U$2.53
- net +12V1: now also U$2.1, U$2.11, U$2.13, U$2.15, U$2.17, U$2.19, U$2.21, U$2.23, U$2.25, U$2.27, U$2.29, U$2.3, U$2.31, U$2.33, U$2.35, U$2.37, U$2.39, U$2.5, U$2.7, U$2.9; no longer SV1.1, SV1.11, SV1.13, SV1.15, SV1.17, SV1.19, SV1.21, SV1.23, SV1.25, SV1.27, SV1.29, SV1.3, SV1.31, SV1.33, SV1.35, SV1.37, SV1.39, SV1.5, SV1.7, SV1.9
- net GND: now also U$2.10, U$2.12, U$2.14, U$2.16, U$2.18, U$2.2, U$2.20, U$2.22, U$2.24, U$2.26, U$2.28, U$2.30, U$2.32, U$2.34, U$2.36, U$2.38, U$2.4, U$2.40, U$2.6, U$2.8; no longer SV1.10, SV1.12, SV1.14, SV1.16, SV1.18, SV1.2, SV1.20, SV1.22, SV1.24, SV1.26, SV1.28, SV1.30, SV1.32, SV1.34, SV1.36, SV1.38, SV1.4, SV1.40, SV1.6, SV1.8
- net N$11: now also U$2.54; no longer JP1.1
- net N$9: now also U$2.52; no longer JP2.1
- net V-: now also U$2.42, U$2.44, U$2.46, U$2.48, U$2.50; no longer SV1.42, SV1.44, SV1.46, SV1.48, SV1.50
- net VCC: now also U$2.41, U$2.43, U$2.45, U$2.47, U$2.49; no longer SV1.41, SV1.43, SV1.45, SV1.47, SV1.49
Other:
- board size 57.4 x 76.2 mm -> 48.3 x 73.7 mm

Commit message: Worked on DC-DC Board layout
Parts:
- removed U$2: POWERBRICKCONNECTOR, newConnector:FE25-2
- added U$3: POWER-BRICK-CONNECTOR, MotherboardParts:POWER-BRICK-CONNECTOR
Connections:
- removed net +12V1: C19.1, C20.1, C21.1, R9.2, U$1.16, U$1.6, U$2.1, U$2.11, U$2.13, U$2.15, U$2.17, U$2.19, U$2.21, U$2.23, U$2.25, U$2.27, U$2.29, U$2.3, U$2.31, U$2.33, U$2.35, U$2.37, U$2.39, U$2.5, U$2.7, U$2.9
- removed net N$11: U$1.10, U$2.54
- new net N$10: U$1.10, U$3.P$53
- new net V+: C19.1, C20.1, C21.1, R9.2, U$1.16, U$1.6, U$3.P$11, U$3.P$12, U$3.P$13, U$3.P$14, U$3.P$15, U$3.P$16, U$3.P$17, U$3.P$18, U$3.P$19, U$3.P$20, U$3.P$21, U$3.P$22, U$3.P$23, U$3.P$24, U$3.P$25, U$3.P$26, U$3.P$27, U$3.P$28, U$3.P$29, U$3.P$30
- net GND: now also U$3.P$31, U$3.P$32, U$3.P$33, U$3.P$34, U$3.P$35, U$3.P$36, U$3.P$37, U$3.P$38, U$3.P$39, U$3.P$40, U$3.P$41, U$3.P$42, U$3.P$43, U$3.P$44, U$3.P$45, U$3.P$46, U$3.P$47, U$3.P$48, U$3.P$49, U$3.P$50, U$3.P$52; no longer U$2.10, U$2.12, U$2.14, U$2.16, U$2.18, U$2.2, U$2.20, U$2.22, U$2.24, U$2.26, U$2.28, U$2.30, U$2.32, U$2.34, U$2.36, U$2.38, U$2.4, U$2.40, U$2.6, U$2.8
- net N$8: now also U$3.P$54; no longer U$2.53
- net N$9: now also U$3.P$51; no longer U$2.52
- net V-: now also U$3.P$10, U$3.P$6, U$3.P$7, U$3.P$8, U$3.P$9; no longer U$2.42, U$2.44, U$2.46, U$2.48, U$2.50
- net VCC: now also U$3.P$1, U$3.P$2, U$3.P$3, U$3.P$4, U$3.P$5; no longer U$2.41, U$2.43, U$2.45, U$2.47, U$2.49
Routing:
- net N$9: track 0.00 -> 75.0 mm
- net N$10: track 0.00 -> 35.9 mm
- net N$8: track 0.00 -> 30.6 mm, vias 0 -> 1
- added copper zone on layer 1, net V+
- removed copper zone on layer 1, net +12V1
Other:
- outline, holes or cut-outs redrawn
