File: DC-DC-Brick/DC-DC-Brick.sch (EAGLE design)
At the start: 20 parts

Commit message: Changes made to DC bricks (see Google Doc)
Parts:
- removed C16: .1uF, rcl:C-USC0603
- removed C19, C20: 15uF, rcl:C-USC3216
- removed C22V1, C22V5, C22V6: EXTENDED_PAD_CAPACITOR, ExtendedPadCap:EXTENDED_PAD_CAPACITOR
- added C1: 1uF, rcl:C-USC0603
- added C3, C4: 220uF, SparkFun-Capacitors:CAP1206
- C15: value .1uF -> 10uF
- renumbered C21 to C2
Connections:
- net GND: now also C1.2; no longer C19.2, C20.2, D1.C
- net N$4: now also D1.C; no longer D1.A
- net N$7: now also U$1.!PG; no longer U$1.PG
- net ON/OFF: now also U$1.ON/!OFF1; no longer U$1.ON/OFF1
- net V+: now also C1.1, D1.A; no longer C19.1, C20.1
- net V-: now also C3.2, C4.2; no longer C16.2, C22V1.4, C22V5.4, C22V6.4
- net VCC: now also C3.1, C4.1; no longer C16.1, C22V1.3, C22V5.3, C22V6.3
Other:
- note added: "10K for first board 22K for second 33K for third"
- note removed: "Removed pulldown res That would cause it to stay on when disconnect"
- moved on the sheet: D1, D2, R4
