File: Power-Conversion.brd (EAGLE design)
At the start: 160 x 81.3 mm, 55 parts, among them J1 AVR_SPI_PRG_6PTH, U1 ATMEGA328P_TQFP, U2 LM1085IS-3.3

Commit message: more routing
Routing:
- net N$31: track 0.00 -> 50.5 mm, vias 0 -> 2
- net N$26: track 0.00 -> 47.0 mm, vias 0 -> 2
- net N$29: track 0.00 -> 35.1 mm, vias 0 -> 1
- net GND: track 11.4 -> 17.7 mm, vias 4 -> 7
Changed lines of the file:
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@@
 <layer number="14" name="Route14" color="1" fill="6" visible="yes" active="yes"/>
 <layer number="15" name="Route15" color="4" fill="6" visible="yes" active="yes"/>
-<layer number="16" name="Bottom" color="1" fill="1" visible="no" active="yes"/>
+<layer number="16" name="Bottom" color="1" fill="1" visible="yes" active="yes"/>
 <layer number="17" name="Pads" color="2" fill="1" visible="yes" active="yes"/>
 <layer number="18" name="Vias" color="2" fill="1" visible="yes" active="yes"/>
@@
 <wire x1="6.01" y1="57.906" x2="6.01" y2="59.223" width="0.4064" layer="1"/>
 <wire x1="6.01" y1="59.223" x2="6.096" y2="59.309" width="0.4064" layer="1"/>
-<wire x1="5.549" y1="40.513" x2="5.588" y2="40.513" width="0.4064" layer="1"/>
-<wire x1="5.588" y1="40.513" x2="6.35" y2="41.275" width="0.4064" layer="1"/>
 <wire x1="6.35" y1="41.275" x2="6.35" y2="42.1704" width="0.4064" layer="1"/>
 <wire x1="6.35" y1="42.1704" x2="6.369" y2="42.1894" width="0.4064" layer="1"/>
@@
 <via x="3.81" y="18.288" extent="1-16" drill="0.4572"/>
 <wire x1="3.81" y1="20.6756" x2="3.81" y2="18.288" width="1.016" layer="1"/>
+<wire x1="5.569" y1="50.7746" x2="5.588" y2="50.7936" width="0.6096" layer="1"/>
+<wire x1="5.588" y1="50.7936" x2="5.588" y2="51.816" width="0.6096" layer="1"/>
+<wire x1="5.588" y1="51.816" x2="5.842" y2="52.07" width="0.6096" layer="1"/>
+<wire x1="5.842" y1="52.07" x2="6.35" y2="52.07" width="0.6096" layer="1"/>
+<wire x1="6.35" y1="52.07" x2="6.858" y2="52.07" width="0.6096" layer="1"/>
+<wire x1="6.858" y1="52.07" x2="7.169" y2="51.759" width="0.6096" layer="1"/>
+<wire x1="7.169" y1="51.759" x2="7.169" y2="50.7746" width="0.6096" layer="1"/>
+<via x="6.35" y="52.07" extent="1-16" drill="0.2032" diameter="0.4572"/>
+<wire x1="6.35" y1="41.275" x2="5.588" y2="40.513" width="0.4064" layer="1"/>
+<wire x1="5.588" y1="40.513" x2="5.549" y2="40.513" width="0.4064" layer="1"/>
+<wire x1="6.369" y1="42.1894" x2="6.35" y2="42.2084" width="0.4064" layer="1"/>
+<wire x1="6.35" y1="42.2084" x2="6.35" y2="43.434" width="0.4064" layer="1"/>
+<via x="6.35" y="43.434" extent="1-16" drill="0.2032" diameter="0.4572"/>
+<via x="6.858" y="39.624" extent="1-16" drill="0.2032" diameter="0.4572"/>
+<wire x1="6.858" y1="39.624" x2="5.588" y2="39.624" width="0.4064" layer="1"/>
 <wire x1="140.97" y1="52.07" x2="146.05" y2="52.07" width="0" layer="19" extent="1-1"/>
 <wire x1="153.67" y1="6.35" x2="153.67" y2="11.43" width="0" layer="19" extent="1-1"/>
 <wire x1="82.55" y1="31.75" x2="87.63" y2="31.75" width="0" layer="19" extent="1-1"/>
-<wire x1="5.569" y1="50.7746" x2="2.794" y2="56.769" width="0" layer="19" extent="1-1"/>
-<wire x1="7.169" y1="50.7746" x2="5.569" y2="50.7746" width="0" layer="19" extent="1-1"/>
-<wire x1="6.369" y1="42.1894" x2="5.569" y2="50.7746" width="0" layer="19" extent="1-1"/>
 </signal>
 <signal name="SCL">
@@
 <contactref element="J1" pad="4"/>
 <contactref element="R6" pad="2"/>
-<wire x1="1.6764" y1="44.482" x2="5.715" y2="54.649" width="0" layer="19" extent="1-1"/>
-<wire x1="5.588" y1="11.684" x2="1.6764" y2="44.482" width="0" layer="19" extent="1-1"/>
+<via x="5.842" y="53.34" extent="1-16" drill="0.2032" diameter="0.4572"/>
+<wire x1="5.715" y1="54.649" x2="5.842" y2="54.649" width="0.4064" layer="1"/>
+<wire x1="5.842" y1="54.649" x2="5.842" y2="53.34" width="0.4064" layer="1"/>
+<via x="3.048" y="45.212" extent="1-16" drill="0.2032" diameter="0.4572"/>
+<wire x1="5.842" y1="53.34" x2="5.842" y2="48.006" width="0.4064" layer="2"/>
+<wire x1="5.842" y1="48.006" x2="3.048" y2="45.212" width="0.4064" layer="2"/>
+<wire x1="2.318" y1="44.482" x2="1.6764" y2="44.482" width="0.4064" layer="1"/>
+<wire x1="3.048" y1="45.212" x2="4.318" y2="43.942" width="0.4064" layer="2"/>
+<wire x1="4.318" y1="43.942" x2="4.318" y2="13.97" width="0.4064" layer="2"/>
+<wire x1="4.318" y1="13.97" x2="5.588" y2="12.7" width="0.4064" layer="2"/>
+<wire x1="5.588" y1="12.7" x2="5.588" y2="11.684" width="0.4064" layer="2"/>
+<wire x1="3.048" y1="45.212" x2="2.318" y2="44.482" width="0.4064" layer="1"/>
 </signal>
 <signal name="N$29">
 <contactref element="J1" pad="1"/>
 <contactref element="U1" pad="16"/>
-<wire x1="3.048" y1="9.144" x2="1.6764" y2="43.682" width="0" layer="19" extent="1-1"/>
+<via x="1.778" y="42.672" extent="1-16" drill="0.2032" diameter="0.4572"/>
+<wire x1="1.6764" y1="43.682" x2="1.778" y2="43.5804" width="0.4064" layer="1"/>
+<wire x1="1.778" y1="43.5804" x2="1.778" y2="42.672" width="0.4064" layer="1"/>
+<wire x1="1.778" y1="42.672" x2="1.778" y2="10.414" width="0.4064" layer="2"/>
+<wire x1="1.778" y1="10.414" x2="3.048" y2="9.144" width="0.4064" layer="2"/>
 </signal>
 <signal name="N$31">
@@
 <contactref element="R5" pad="2"/>
 <contactref element="U1" pad="17"/>
-<wire x1="3.169" y1="42.1894" x2="4.318" y2="54.649" width="0" layer="19" extent="1-1"/>
-<wire x1="5.588" y1="9.144" x2="3.169" y2="42.1894" width="0" layer="19" extent="1-1"/>
+<via x="4.572" y="53.34" extent="1-16" drill="0.2032" diameter="0.4572"/>
+<wire x1="4.318" y1="54.649" x2="4.572" y2="54.649" width="0.4064" layer="1"/>
+<wire x1="4.572" y1="54.649" x2="4.572" y2="53.34" width="0.4064" layer="1"/>
+<via x="3.302" y="43.942" extent="1-16" drill="0.2032" diameter="0.4572"/>
+<wire x1="4.572" y1="53.34" x2="2.032" y2="50.8" width="0.4064" layer="2"/>
+<wire x1="2.032" y1="50.8" x2="2.032" y2="44.45" width="0.4064" layer="2"/>
+<wire x1="2.032" y1="44.45" x2="2.54" y2="43.942" width="0.4064" layer="2"/>
+<wire x1="2.54" y1="43.942" x2="3.302" y2="43.942" width="0.4064" layer="2"/>
+<wire x1="3.302" y1="43.942" x2="3.302" y2="13.462" width="0.4064" layer="2"/>
+<wire x1="3.302" y1="13.462" x2="4.318" y2="12.446" width="0.4064" layer="2"/>
+<wire x1="4.318" y1="12.446" x2="4.318" y2="10.414" width="0.4064" layer="2"/>
+<wire x1="4.318" y1="10.414" x2="5.588" y2="9.144" width="0.4064" layer="2"/>
+<wire x1="3.302" y1="43.942" x2="3.169" y2="43.809" width="0.4064" layer="1"/>
+<wire x1="3.169" y1="43.809" x2="3.169" y2="42.1894" width="0.4064" layer="1"/>
 </signal>
 <signal name="N$27">

Commit message: layer stackup+more routing
Routing:
- net N$27: track 0.00 -> 11.4 mm, vias 0 -> 2
- net N$19: vias 2 -> 1
Changed lines of the file:
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@@
 <setting verticaltext="up"/>
 </settings>
-<grid distance="10" unitdist="mil" unit="mil" style="dots" multiple="1" display="yes" altdistance="0.025" altunitdist="inch" altunit="inch"/>
+<grid distance="5" unitdist="mil" unit="mil" style="dots" multiple="1" display="yes" altdistance="0.025" altunitdist="inch" altunit="inch"/>
 <layers>
 <layer number="1" name="Top" color="4" fill="1" visible="yes" active="yes"/>
 <layer number="2" name="Route2" color="1" fill="3" visible="yes" active="yes"/>
-<layer number="3" name="Route3" color="4" fill="3" visible="yes" active="yes"/>
-<layer number="14" name="Route14" color="1" fill="6" visible="yes" active="yes"/>
+<layer number="3" name="Route3" color="4" fill="3" visible="no" active="no"/>
+<layer number="14" name="Route14" color="1" fill="6" visible="no" active="no"/>
 <layer number="15" name="Route15" color="4" fill="6" visible="yes" active="yes"/>
 <layer number="16" name="Bottom" color="1" fill="1" visible="yes" active="yes"/>
@@
 </class>
 </classes>
-<designrules name="default">
+<designrules name="default *">
 <description language="de">&lt;b&gt;EAGLE Design Rules&lt;/b&gt;
 &lt;p&gt;
@@
 necessary adjustments and save your customized
 design rules under a new name.</description>
-<param name="layerSetup" value="(1*16)"/>
+<param name="layerSetup" value="(1*2*15*16)"/>
 <param name="mtCopper" value="0.035mm 0.035mm 0.035mm 0.035mm 0.035mm 0.035mm 0.035mm 0.035mm 0.035mm 0.035mm 0.035mm 0.035mm 0.035mm 0.035mm 0.035mm 0.035mm"/>
 <param name="mtIsolate" value="1.5mm 0.15mm 0.2mm 0.15mm 0.2mm 0.15mm 0.2mm 0.15mm 0.2mm 0.15mm 0.2mm 0.15mm 0.2mm 0.15mm 0.2mm"/>
 <param name="mdWireWire" value="8mil"/>
 <param name="mdWirePad" value="8mil"/>
-<param name="mdWireVia" value="8mil"/>
+<param name="mdWireVia" value="6mil"/>
 <param name="mdPadPad" value="8mil"/>
-<param name="mdPadVia" value="8mil"/>
-<param name="mdViaVia" value="8mil"/>
-<param name="mdSmdPad" value="8mil"/>
-<param name="mdSmdVia" value="8mil"/>
+<param name="mdPadVia" value="6mil"/>
+<param name="mdViaVia" value="6mil"/>
+<param name="mdSmdPad" value="6mil"/>
+<param name="mdSmdVia" value="6mil"/>
 <param name="mdSmdSmd" value="8mil"/>
 <param name="mdViaViaSameLayer" value="8mil"/>
@@
 <param name="mdSmdStop" value="0mil"/>
 <param name="msWidth" value="10mil"/>
-<param name="msDrill" value="24mil"/>
+<param name="msDrill" value="6mil"/>
 <param name="msMicroVia" value="9.99mm"/>
 <param name="msBlindViaRatio" value="0.5"/>
@@
 <vertex x="55.88" y="7.62"/>
 </polygon>
-<via x="2.413" y="67.818" extent="1-16" drill="0.2032"/>
-<wire x1="2.413" y1="67.818" x2="2.413" y2="66.89" width="0.4064" layer="1"/>
-<via x="2.794" y="56.769" extent="1-16" drill="0.2032"/>
-<wire x1="2.76" y1="57.906" x2="2.76" y2="56.803" width="0.4064" layer="1"/>
-<wire x1="2.76" y1="56.803" x2="2.794" y2="56.769" width="0.4064" layer="1"/>
+<via x="2.413" y="68.072" extent="1-16" drill="0.2032"/>
+<wire x1="2.413" y1="68.072" x2="2.413" y2="66.89" width="0.4064" layer="1"/>
+<via x="2.667" y="56.261" extent="1-16" drill="0.2032"/>
+<wire x1="2.76" y1="57.906" x2="2.76" y2="56.422" width="0.4064" layer="1"/>
+<wire x1="2.76" y1="56.422" x2="2.667" y2="56.261" width="0.4064" layer="1"/>
 <via x="6.096" y="59.309" extent="1-16" drill="0.2032"/>
 <wire x1="6.01" y1="57.906" x2="6.01" y2="59.223" width="0.4064" layer="1"/>
@@
 <wire x1="6.35" y1="42.1704" x2="6.369" y2="42.1894" width="0.4064" layer="1"/>
 <wire x1="5.549" y1="40.513" x2="5.549" y2="38.862" width="0.4064" layer="1"/>
-<via x="3.81" y="18.288" extent="1-16" drill="0.4572"/>
-<wire x1="3.81" y1="20.6756" x2="3.81" y2="18.288" width="1.016" layer="1"/>
-<wire x1="5.569" y1="50.7746" x2="5.588" y2="50.7936" width="0.6096" layer="1"/>
-<wire x1="5.588" y1="50.7936" x2="5.588" y2="51.816" width="0.6096" layer="1"/>
-<wire x1="5.588" y1="51.816" x2="5.842" y2="52.07" width="0.6096" layer="1"/>
-<wire x1="5.842" y1="52.07" x2="6.35" y2="52.07" width="0.6096" layer="1"/>
-<wire x1="6.35" y1="52.07" x2="6.858" y2="52.07" width="0.6096" layer="1"/>
-<wire x1="6.858" y1="52.07" x2="7.169" y2="51.759" width="0.6096" layer="1"/>
-<wire x1="7.169" y1="51.759" x2="7.169" y2="50.7746" width="0.6096" layer="1"/>
-<via x="6.35" y="52.07" extent="1-16" drill="0.2032" diameter="0.4572"/>
+<via x="2.54" y="20.701" extent="1-16" drill="0.2032"/>
+<wire x1="3.81" y1="20.6756" x2="2.54" y2="20.701" width="1.016" layer="1"/>
+<wire x1="5.569" y1="50.7746" x2="5.588" y2="50.7936" width="0.508" layer="1"/>
+<wire x1="5.588" y1="50.7936" x2="5.588" y2="51.816" width="0.508" layer="1"/>
+<wire x1="5.588" y1="51.816" x2="5.842" y2="52.07" width="0.508" layer="1"/>
+<wire x1="5.842" y1="52.07" x2="6.731" y2="52.07" width="0.508" layer="1"/>
+<wire x1="6.731" y1="52.07" x2="6.858" y2="52.07" width="0.508" layer="1"/>
+<wire x1="6.858" y1="52.07" x2="7.169" y2="51.759" width="0.508" layer="1"/>
+<wire x1="7.169" y1="51.759" x2="7.169" y2="50.7746" width="0.508" layer="1"/>
+<via x="6.731" y="52.07" extent="1-16" drill="0.2032" diameter="0.4572"/>
 <wire x1="6.35" y1="41.275" x2="5.588" y2="40.513" width="0.4064" layer="1"/>
 <wire x1="5.588" y1="40.513" x2="5.549" y2="40.513" width="0.4064" layer="1"/>
@@
 <wire x1="2.76" y1="65.19" x2="2.76" y2="63.506" width="0.4064" layer="1"/>
 <wire x1="4.06" y1="63.506" x2="4.06" y2="62.353" width="0.4064" layer="1"/>
-<wire x1="4.06" y1="62.353" x2="3.937" y2="62.23" width="0.4064" layer="1"/>
-<wire x1="2.921" y1="62.23" x2="2.794" y2="62.357" width="0.4064" layer="1"/>
+<wire x1="4.06" y1="62.353" x2="3.937" y2="62.103" width="0.4064" layer="1"/>
+<wire x1="2.921" y1="62.103" x2="2.794" y2="62.357" width="0.4064" layer="1"/>
 <wire x1="2.794" y1="62.357" x2="2.794" y2="63.472" width="0.4064" layer="1"/>
 <wire x1="2.794" y1="63.472" x2="2.76" y2="63.506" width="0.4064" layer="1"/>
@@
 <vertex x="5.461" y="43.18"/>
 </polygon>
-<wire x1="3.937" y1="62.23" x2="2.921" y2="62.23" width="0.6096" layer="1"/>
-<wire x1="2.921" y1="62.23" x2="1.778" y2="61.087" width="0.6096" layer="1"/>
-<wire x1="1.778" y1="61.087" x2="1.778" y2="54.8132" width="0.6096" layer="1"/>
+<wire x1="3.937" y1="62.103" x2="2.921" y2="62.103" width="0.6096" layer="1"/>
+<wire x1="2.921" y1="62.103" x2="1.778" y2="60.96" width="0.6096" layer="1"/>
+<wire x1="1.778" y1="60.96" x2="1.778" y2="54.8132" width="0.6096" layer="1"/>
 <wire x1="1.778" y1="54.8132" x2="4.7752" y2="51.816" width="0.6096" layer="1"/>
 <wire x1="4.7752" y1="51.816" x2="4.7752" y2="50.8446" width="0.6096" layer="1"/>
@@
 <contactref element="U$8" pad="P$11"/>
 <contactref element="I2C_ESC5" pad="1"/>
-<via x="9.271" y="56.007" extent="1-16" drill="0.2032" diameter="0.4572"/>
 <wire x1="9.26" y1="57.906" x2="9.26" y2="56.018" width="0.3048" layer="1"/>
 <wire x1="9.26" y1="56.018" x2="9.271" y2="56.007" width="0.3048" layer="1"/>
 <via x="9.26" y="56.018" extent="1-16" drill="0.2032" diameter="0.4572"/>
-<wire x1="9.26" y1="56.018" x2="11.303" y2="53.975" width="0.3048" layer="2"/>
 <wire x1="11.303" y1="53.975" x2="11.303" y2="40.767" width="0.3048" layer="2"/>
 <wire x1="11.303" y1="40.767" x2="13.97" y2="38.1" width="0.3048" layer="2"/>
+<wire x1="9.26" y1="56.018" x2="11.303" y2="53.975" width="0.3048" layer="2"/>
 </signal>
 <signal name="N$20">
@@
 <wire x1="5.842" y1="53.34" x2="5.842" y2="48.006" width="0.4064" layer="2"/>
 <wire x1="5.842" y1="48.006" x2="3.048" y2="45.212" width="0.4064" layer="2"/>
-<wire x1="2.318" y1="44.482" x2="1.6764" y2="44.482" width="0.4064" layer="1"/>
+<wire x1="2.445" y1="44.482" x2="1.6764" y2="44.482" width="0.4064" layer="1"/>
 <wire x1="3.048" y1="45.212" x2="4.318" y2="43.942" width="0.4064" layer="2"/>
 <wire x1="4.318" y1="43.942" x2="4.318" y2="13.97" width="0.4064" layer="2"/>
 <wire x1="4.318" y1="13.97" x2="5.588" y2="12.7" width="0.4064" layer="2"/>
 <wire x1="5.588" y1="12.7" x2="5.588" y2="11.684" width="0.4064" layer="2"/>
-<wire x1="3.048" y1="45.212" x2="2.318" y2="44.482" width="0.4064" layer="1"/>
+<wire x1="3.048" y1="45.212" x2="2.445" y2="44.482" width="0.4064" layer="1"/>
 </signal>
 <signal name="N$29">
@@
 <contactref element="U1" pad="11"/>
 <contactref element="U$8" pad="P$2"/>
-<wire x1="1.6764" y1="47.682" x2="3.41" y2="57.906" width="0" layer="19" extent="1-1"/>
+<wire x1="1.6764" y1="47.682" x2="2.47" y2="47.682" width="0.4064" layer="1"/>
+<wire x1="2.47" y1="47.682" x2="2.794" y2="48.006" width="0.4064" layer="1"/>
+<via x="2.794" y="48.006" extent="1-16" drill="0.2032" diameter="0.4572"/>
+<wire x1="2.794" y1="48.006" x2="2.794" y2="55.118" width="0.4064" layer="15"/>
+<via x="2.794" y="55.118" extent="1-16" drill="0.2032" diameter="0.4572"/>
+<wire x1="2.794" y1="55.118" x2="3.41" y2="55.734" width="0.4064" layer="1"/>
+<wire x1="3.41" y1="55.734" x2="3.41" y2="57.906" width="0.4064" layer="1"/>
 </signal>
 </signals>

Commit message: More routing
Routing:
- net GSCLK: track 0.00 -> 19.3 mm, vias 0 -> 2
Changed lines of the file:
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@@
 <contactref element="U1" pad="13"/>
 <contactref element="U$8" pad="P$25"/>
-<wire x1="1.6764" y1="46.082" x2="4.71" y2="63.506" width="0" layer="19" extent="1-1"/>
+<wire x1="4.71" y1="63.506" x2="4.699" y2="63.506" width="0.254" layer="1"/>
+<wire x1="4.699" y1="63.506" x2="4.699" y2="62.103" width="0.254" layer="1"/>
+<wire x1="4.699" y1="62.103" x2="4.699" y2="55.88" width="0.254" layer="15"/>
+<wire x1="4.699" y1="55.88" x2="3.683" y2="54.864" width="0.254" layer="15"/>
+<wire x1="3.683" y1="54.864" x2="3.683" y2="47.117" width="0.254" layer="15"/>
+<via x="4.699" y="62.103" extent="1-16" drill="0.2032" diameter="0.4572"/>
+<via x="3.683" y="47.117" extent="1-16" drill="0.2032" diameter="0.4572"/>
+<wire x1="3.683" y1="47.117" x2="2.648" y2="46.082" width="0.254" layer="1"/>
+<wire x1="2.648" y1="46.082" x2="1.6764" y2="46.082" width="0.254" layer="1"/>
 </signal>
 <signal name="N$25">
