File: Power-Conversion.sch (EAGLE design)
At the start: 113 parts, among them T3 FDN340P, U1 ATMEGA328P_TQFP, U4 PCA9685, U5 FT232RLSSOP, U7 LM2678

Commit message: stuff
Parts:
- added LED5, LED6: Red, SparkFun:LED0603
- added R12, R13: 470, resistor:R-US_R0603
- added RN1, RN2: (no value), resistor-dil:4R-N0603-ARC
Connections:
- new net A0: RN1A.1, U4.A0
- new net A1: RN1B.1, U4.A1
- new net A2: RN1C.1, U4.A2
- new net A3: RN1D.1, U4.A3
- new net A4: RN2A.1, U4.A4
- new net A5: RN2B.1, U4.A5
- new net LED1: R12.2, U1.PD3(INT1)
- new net LED2: R13.2, U1.PD4(XCK/T0)
- new net N$41: LED5.A, R12.1
- new net N$42: LED6.A, R13.1
- net GND: now also LED5.C, LED6.C, RN1A.2, RN1B.2, RN1C.2, RN1D.2, RN2A.2, RN2B.2, RN2C.2, RN2D.2; no longer U4.A0, U4.A1, U4.A2, U4.A3, U4.A4, U4.A5
